File: ESP32-Small-SRWLED/ESP32-Small-SRWLED/ESP32-Small-SRWLED.kicad_pcb (KiCad board)
At the start: 4 copper layers, 19.6 x 20.3 mm, 35 parts, among them J1 Conn_01x07, J2 Conn_02x05_Odd_Even_MountingP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, J3 Conn_01x05, U1 TPS54202DDC, U10 AO3400A, U2 MSM261D4030H1CPM, U3 ESP32-WROOM-32D, U4 AO3400A, U5 AO3400A, U6 AO3400A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

Commit message: edited website link
Other:
- board text added: "wszeto9. github.io /smolwled"
- board text removed: "ESP32 Small SRWLED RevA Winnie Szeto"
Changed lines of the file:
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@@
   (gr_arc (start 124.9 84.499998) (mid 124.617158 84.38284) (end 124.5 84.099998) (layer "Edge.Cuts") (width 0.1))
   (gr_line (start 124.500002 64.6) (end 124.5 84.099998) (layer "Edge.Cuts") (width 0.1))
-  (gr_text "ESP32 Small \nSRWLED RevA\nWinnie Szeto" (at 125.5 83.1 270) (layer "F.Cu")
-    (effects (font (size 0.25 0.25) (thickness 0.0625)))
+  (gr_text "wszeto9.\ngithub.io\n/smolwled" (at 125.5 83.1 270) (layer "F.Cu")
+    (effects (font (size 0.3 0.3) (thickness 0.075)))
   )
   (gr_text "ESP32 Small SRWLED\nRev A\nWinnie Szeto\ngithub.com/wszeto9" (at 134.5 67.8) (layer "B.SilkS")
