File: ESP32-Small-SRWLED/ESP32-Small-SRWLED/ESP32-Small-SRWLED.kicad_sch (KiCad schematic)
At the start: 34 parts, among them J1 Conn_01x02, J2 Conn_02x05_Odd_Even_MountingP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, J3 Conn_01x05, U1 TPS54202DDC, U10 AO3400A, U2 MSM261D4030H1CPM, U3 ESP32-WROOM-32D, U4 AO3400A, U5 AO3400A, U6 AO3400A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

Commit message: edited website link
Parts:
- removed J1: Conn_01x02, Connector_JST:JST_PH_B2B-PH-SM4-TB_1x02-1MP_P2.00mm_Vertical, symbol Connector_Generic:Conn_01x02
- removed J?: Conn_01x05, WS_LCSC_Connectors:1x5 solder pad, symbol Connector_Generic:Conn_01x05
- added D1: LED_White, LED_SMD:LED_0603_1608Metric, symbol WS_LCSC_Optoelectronics:LED_White
- added J1: Conn_01x07, WS_LCSC_Connectors:1x7 wire solder pad, symbol Connector_Generic:Conn_01x07
- added R9: 0402,220, R_0402_1005Metric, symbol jlcpcb-basic-resistor:0402,220
Connections:
- net 3V3: now also D1.2 (A)
- net ADDR1_SHIFTED: now also J1.4 (Pin_4)
- net ADDR2_SHIFTED: now also J1.6 (Pin_6)
- net GND: now also J1.2 (Pin_2), J1.3 (Pin_3), J1.7 (Pin_7)
- net G_SIG: now also U3.27 (IO16); no longer U3.28 (IO17)
- net R_SIG: now also U3.28 (IO17); no longer U3.29 (IO5)
- net VIN: now also J1.1 (Pin_1), J1.5 (Pin_5)
- net at U3.9 (IO33): now also R9.2
- new net: D1.1 (K), R9.1
