File: PCB/ESP32-Small-SRWLED.kicad_sch (KiCad schematic)
At the start: 35 parts, among them J1 Conn_01x07, J2 Conn_02x05_Odd_Even_MountingP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, J3 Conn_01x05, U1 TPS54202DDC, U10 AO3400A, U2 MSM261D4030H1CPM, U3 ESP32-WROOM-32D, U4 AO3400A, U5 AO3400A, U6 AO3400A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

Commit message: sent to fab
Parts:
- J1: value Conn_01x07 -> SolderHeader1x7
- J2: value Conn_02x05_Odd_Even_MountingPin -> BB10-10S-02; LCSC C2763970 -> C2763962
- J3: value Conn_01x05 -> SolderHeader1x5
- U10, U4, U5, U6, U7, U9: LCSC C20917 -> C700953
- U3: LCSC (none) -> C473005
- U8: value L78L05_SOT89 -> 78L05G-AB3-R
Connections:
- net SW: no longer C4.2, L1.1, U1.2 (SW)
- new net: C4.2, L1.1, U1.2 (SW)
Other:
- note added: "5V LDO for 5V Logic Level Shifting"
- note added: "Addressible 3.3V to 5V Logic Level Shifter"
- note added: "Analog RGBW Driver"
- note added: "CHANGELOG/NOTES REV A: Initial Design. Runs Analog and Addressible lights off 5-24V"
- note added: "ESP32"
- note added: "PDM Mic"
- note added: "Programming header"
- note added: "Soldered wire pads"
- note added: "VIN to 3.3V Buck Converter"
- note removed: "CHANGELOG/NOTES REV A:"
- moved on the sheet: C1, C10, C11, C2, C3, C4, C5, C6, C7, C8, C9, D1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
