File: PCB/ESP32-Small-SRWLED.kicad_pcb (KiCad board)
At the start: 4 copper layers, 19.6 x 20.3 mm, 35 parts, among them J1 Conn_01x07, J2 Conn_02x05_Odd_Even_MountingP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, J3 Conn_01x05, U1 TPS54202DDC, U10 AO3400A, U2 MSM261D4030H1CPM, U3 ESP32-WROOM-32D, U4 AO3400A, U5 AO3400A, U6 AO3400A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

Commit message: sent to fab
Parts:
- J1: value Conn_01x07 -> SolderHeader1x7
- J2: value Conn_02x05_Odd_Even_MountingPin -> BB10-10S-02
- J3: value Conn_01x05 -> SolderHeader1x5
- U8: value L78L05_SOT89 -> 78L05G-AB3-R
Connections:
- net /SW renamed Net-(C4-Pad2)
Routing:
- net /GND: vias 51 -> 50
Other:
- board text added: "B"
Changed lines of the file:
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@@
   (net 3 "/VIN")
   (net 4 "Net-(C4-Pad1)")
-  (net 5 "/SW")
+  (net 5 "Net-(C4-Pad2)")
   (net 6 "/3V3")
   (net 7 "Net-(C5-Pad2)")
@@
   (net 49 "/ADDR2_SHIFTED")
   (net 50 "Net-(D1-Pad1)")
-  (net 51 "Net-(U3-Pad9)")
+  (net 51 "Net-(R9-Pad2)")
   (footprint "Capacitor_SMD:C_0402_1005Metric" (layer "F.Cu")
     (at 132.4 70.45 90)
@@
     (at 134.316772 66.70536)
     (descr "YXT-BB10-10S-02")
-    (property "LCSC" "C2763970")
+    (property "LCSC" "C2763962")
     (property "Sheetfile" "ESP32-Small-SRWLED.kicad_sch")
     (property "Sheetname" "")
@@
       (effects (font (size 0.8 0.8) (thickness 0.12)))
     )
-    (fp_text value "Conn_02x05_Odd_Even_MountingPin" (at 0 2.7) (layer "F.Fab")
+    (fp_text value "BB10-10S-02" (at 0 2.7) (layer "F.Fab")
       (effects (font (size 1 1) (thickness 0.15)))
     )
@@
     (descr "SOT, 3 Pin (https://www.jedec.org/system/files/docs/to-236h.pdf variant AB), generated with kicad-footprint-generator ipc_gullwing_generator.py")
     (tags "SOT TO_SOT_SMD")
-    (property "LCSC" "C20917")
+    (property "LCSC" "C700953")
     (property "Sheetfile" "ESP32-Small-SRWLED.kicad_sch")
     (property "Sheetname" "")
@@
     (descr "SOT, 3 Pin (https://www.jedec.org/system/files/docs/to-236h.pdf variant AB), generated with kicad-footprint-generator ipc_gullwing_generator.py")
     (tags "SOT TO_SOT_SMD")
-    (property "LCSC" "C20917")
+    (property "LCSC" "C700953")
     (property "Sheetfile" "ESP32-Small-SRWLED.kicad_sch")
     (property "Sheetname" "")
@@
       (net 2 "/GND") (pinfunction "GND") (pintype "power_in"))
     (pad "2" smd roundrect (at -1.1375 0 270) (size 1.325 0.6) (layers "F.Cu" "F.Paste" "F.Mask") (roundrect_rratio 0.25)
-      (net 5 "/SW") (pinfunction "SW") (pintype "power_out"))
+      (net 5 "Net-(C4-Pad2)") (pinfunction "SW") (pintype "power_out"))
     (pad "3" smd roundrect (at -1.1375 0.95 270) (size 1.325 0.6) (layers "F.Cu" "F.Paste" "F.Mask") (roundrect_rratio 0.25)
       (net 3 "/VIN") (pinfunction "VIN") (pintype "power_in"))
@@
     (descr "SOT, 3 Pin (https://www.jedec.org/system/files/docs/to-236h.pdf variant AB), generated with kicad-footprint-generator ipc_gullwing_generator.py")
     (tags "SOT TO_SOT_SMD")
-    (property "LCSC" "C20917")
+    (property "LCSC" "C700953")
     (property "Sheetfile" "ESP32-Small-SRWLED.kicad_sch")
     (property "Sheetname" "")
@@
     (fp_line (start 2 2) (end 2 -2) (layer "F.Fab") (width 0.1))
     (pad "1" smd rect (at -1.185 0 90) (size 0.98 3.7) (layers "F.Cu" "F.Paste" "F.Mask")
-      (net 5 "/SW") (pintype "passive"))
+      (net 5 "Net-(C4-Pad2)") (pintype "passive"))
     (pad "2" smd rect (at 1.185 0 90) (size 0.98 3.7) (layers "F.Cu" "F.Paste" "F.Mask")
       (net 6 "/3V3") (pintype "passive"))
@@
       (effects (font (size 1 1) (thickness 0.15)))
     )
-    (fp_text value "L78L05_SOT89" (at 0.3 3.5 90) (layer "F.Fab")
+    (fp_text value "78L05G-AB3-R" (at 0.3 3.5 90) (layer "F.Fab")
       (effects (font (size 1 1) (thickness 0.15)))
     )
@@
     (descr "SOT, 3 Pin (https://www.jedec.org/system/files/docs/to-236h.pdf variant AB), generated with kicad-footprint-generator ipc_gullwing_generator.py")
     (tags "SOT TO_SOT_SMD")
-    (property "LCSC" "C20917")
+    (property "LCSC" "C700953")
     (property "Sheetfile" "ESP32-Small-SRWLED.kicad_sch")
     (property "Sheetname" "")
@@
     (descr "SOT, 3 Pin (https://www.jedec.org/system/files/docs/to-236h.pdf variant AB), generated with kicad-footprint-generator ipc_gullwing_generator.py")
     (tags "SOT TO_SOT_SMD")
-    (property "LCSC" "C20917")
+    (property "LCSC" "C700953")
     (property "Sheetfile" "ESP32-Small-SRWLED.kicad_sch")
     (property "Sheetname" "")
@@
       (effects (font (size 1 1) (thickness 0.15)))
     )
-    (fp_text value "Conn_01x07" (at 0 1 unlocked) (layer "F.Fab")
+    (fp_text value "SolderHeader1x7" (at 0 1 unlocked) (layer "F.Fab")
       (effects (font (size 1 1) (thickness 0.15)))
     )
@@
       (net 4 "Net-(C4-Pad1)") (pintype "passive"))
     (pad "2" smd roundrect (at 0.48 0 270) (size 0.56 0.62) (layers "F.Cu" "F.Paste" "F.Mask") (roundrect_rratio 0.25)
-      (net 5 "/SW") (pintype "passive"))
+      (net 5 "Net-(C4-Pad2)") (pintype "passive"))
     (model "${KICAD6_3DMODEL_DIR}/Capacitor_SMD.3dshapes/C_0402_1005Metric.wrl"
       (offset (xyz 0 0 0))
@@
       (net 50 "Net-(D1-Pad1)") (pintype "passive"))
     (pad "2" smd roundrect (at 0.51 0 270) (size 0.54 0.64) (layers "F.Cu" "F.Paste" "F.Mask") (roundrect_rratio 0.25)
-      (net 51 "Net-(U3-Pad9)") (pintype "passive"))
+      (net 51 "Net-(R9-Pad2)") (pintype "passive"))
     (model "${KICAD6_3DMODEL_DIR}/Resistor_SMD.3dshapes/R_0402_1005Metric.wrl"
       (offset (xyz 0 0 0))
@@
     (descr "SOT, 3 Pin (https://www.jedec.org/system/files/docs/to-236h.pdf variant AB), generated with kicad-footprint-generator ipc_gullwing_generator.py")
     (tags "SOT TO_SOT_SMD")
-    (property "LCSC" "C20917")
+    (property "LCSC" "C700953")
     (property "Sheetfile" "ESP32-Small-SRWLED.kicad_sch")
     (property "Sheetname" "")
@@
       (effects (font (size 1 1) (thickness 0.15)))
     )
-    (fp_text value "Conn_01x05" (at 0 3.8 90) (layer "F.Fab")
+    (fp_text value "SolderHeader1x5" (at 0 3.8 90) (layer "F.Fab")
       (effects (font (size 1 1) (thickness 0.15)))
     )
@@
     (descr "Single 2.4 GHz Wi-Fi and Bluetooth combo chip https://www.espressif.com/sites/default/files/documentation/esp32-wroom-32_datasheet_en.pdf")
     (tags "Single 2.4 GHz Wi-Fi and Bluetooth combo  chip")
+    (property "LCSC" "C473005")
     (property "Sheetfile" "ESP32-Small-SRWLED.kicad_sch")
     (property "Sheetname" "")
@@
       (net 26 "unconnected-(U3-Pad8)") (pinfunction "IO32") (pintype "bidirectional"))
     (pad "9" smd rect (at -8.5 -1.905 180) (size 2 0.9) (layers "B.Cu" "B.Paste" "B.Mask")
-      (net 51 "Net-(U3-Pad9)") (pinfunction "IO33") (pintype "bidirectional"))
+      (net 51 "Net-(R9-Pad2)") (pinfunction "IO33") (pintype "bidirectional"))
     (pad "10" smd rect (at -8.5 -3.175 180) (size 2 0.9) (layers "B.Cu" "B.Paste" "B.Mask")
       (net 41 "/ADDR2") (pinfunction "IO25") (pintype "bidirectional"))
@@
   (gr_line (start 136.5 84.3) (end 136.5 80.2) (layer "F.SilkS") (width 0.12))
   (gr_line (start 138.996359 80.2) (end 139 84.3) (layer "F.SilkS") (width 0.12))
-  (gr_line (start 128.8 79.85) (end 128.8 84.3) (layer "F.SilkS") (width 0.12))
+  (gr_line (start 128.8 80.05) (end 128.8 84.3) (layer "F.SilkS") (width 0.12))
   (gr_line (start 141.6 84.3) (end 141.6 80.2) (layer "F.SilkS") (width 0.12))
   (gr_line (start 129.25 68.565) (end 124.7 68.55) (layer "F.SilkS") (width 0.12))
@@
     (effects (font (size 0.77 0.77) (thickness 0.12)))
   )
+  (gr_text "B\n" (at 128.5 69.2) (layer "F.SilkS")
+    (effects (font (size 0.8 0.8) (thickness 0.12)))
+  )
   (gr_text "G" (at 128.5 76.05) (layer "F.SilkS")
     (effects (font (size 0.8 0.8) (thickness 0.12)))
@@
     (effects (font (size 0.8 0.8) (thickness 0.12)))
   )
-  (gr_text "IO33" (at 140.05 64.9) (layer "F.SilkS")
+  (gr_text "IO33" (at 140.2 64.9) (layer "F.SilkS")
     (effects (font (size 0.8 0.8) (thickness 0.12)))
   )
@@
   (via (at 132.1 68.9) (size 0.45) (drill 0.25) (layers "F.Cu" "B.Cu") (free) (net 2))
   (via (at 130.4 73.3) (size 0.45) (drill 0.25) (layers "F.Cu" "B.Cu") (free) (net 2))
-  (via (at 136.35 71.3) (size 0.45) (drill 0.25) (layers "F.Cu" "B.Cu") (net 2))
   (via (at 134.5 77.3) (size 0.45) (drill 0.25) (layers "F.Cu" "B.Cu") (net 2))
   (via (at 134.85 68.775) (size 0.45) (drill 0.2) (layers "F.Cu" "B.Cu") (free) (net 2))
@@
   (via (at 128.55 65.5) (size 0.45) (drill 0.25) (layers "F.Cu" "B.Cu") (free) (net 2))
   (via (at 129.5 81.6) (size 0.45) (drill 0.25) (layers "F.Cu" "B.Cu") (net 2))
-  (via (at 133.55 72.575) (size 0.45) (drill 0.2) (layers "F.Cu" "B.Cu") (net 2))
+  (via (at 133.4 72.8) (size 0.45) (drill 0.2) (layers "F.Cu" "B.Cu") (net 2))
   (via (at 133.1 81.4) (size 0.45) (drill 0.25) (layers "F.Cu" "B.Cu") (net 2))
   (via (at 134.4 76.5) (size 0.45) (drill 0.25) (layers "F.Cu" "B.Cu") (net 2))
@@
     )
   )
-  (zone (net 5) (net_name "/SW") (layer "F.Cu") (hatch edge 0.508)
+  (zone (net 5) (net_name "Net-(C4-Pad2)") (layer "F.Cu") (hatch edge 0.508)
     (priority 2)
     (connect_pads yes (clearance 0.2))

Commit message: Adding documentation
Other:
- board text added: "16"
- board text added: "GND 26 +V 25 GND"
- board text removed: "18"
- board text removed: "GND 25 +V 26 GND"
